File: Schraeg/Schraeg.sch (KiCad schematic (older format))
At the start: 56 parts, among them U1 TL074, U2 TL074, U3 V2164

Commit message: Corrected alignment between panel and pcb, changed to slide switches, trimpot for resonance (leaves more space for cutoff) and new panel design.
Parts:
- removed AUDIO_IN1, BP_OUT1, FM_IN1, HP_OUT1, LP_OUT1, RES_CV1, V_OCT_IN1: PJ301M-12, Eurocad:PJ301M-12, symbol eurocad:PJ301M-12
- added J1, J2, J3, J4, J5, J6, J7: PJ398SM, barullo_eurorack:Jack_3.5mm_QingPu_WQP-PJ398SM_Vertical_CircularHoles, symbol Connector:AudioJack2_SwitchT
- CUTOFF1: footprint Eurocad:Alpha9mmPot -> barullo_eurorack:Potentiometer_Alps-Alpha-Bourns_Single_Vertical
- FM_ATTV1, INPUT_GAIN1, RESONANCE1, RES_ATTV1: footprint Eurocad:Alpha9mmPot -> barullo_eurorack:Potentiometer_Trimmer_9mm_Vertical
- SW_DRIVE1, SW_RES_DIST1, SW_WOBBLE1: footprint Connector_PinHeader_2.54mm:PinHeader_1x03_P2.54mm_Vertical -> barullo_eurorack:SW_NKK_CS1xA
- U3: symbol v2164:V2164 -> Schraeg-rescue:V2164-v2164
Connections:
- wire segments 178 -> 179
Other:
- moved on the sheet: C2

Commit message: Changed power symbol to generic connector
Parts:
- U3: symbol Schraeg-rescue:V2164-v2164 -> Schraeg-rescue:V2164-v2164-Schraeg-rescue
Changed lines of the file:
@@
 	4900 2650 5100 2650
 $Comp
-L Schraeg-rescue:V2164-v2164 U3
+L Schraeg-rescue:V2164-v2164-Schraeg-rescue U3
 U 1 1 5D5C12B5
 P 4700 3950

Commit message: V2164 symbol in a new library to avoid missing dependencies.
Parts:
- removed U3: V2164, Package_SO:SOIC-16_3.9x9.9mm_P1.27mm, symbol Schraeg-rescue:V2164-v2164-Schraeg-rescue
- added U3: V2164, Package_SO:SOIC-16_3.9x9.9mm_P1.27mm, symbol Schraeg:V2164
Connections:
- wire segments 179 -> 178
Changed lines of the file:
@@
 	4900 2650 5100 2650
-$Comp
-L Schraeg-rescue:V2164-v2164-Schraeg-rescue U3
-U 1 1 5D5C12B5
-P 4700 3950
-AR Path="/5D5C12B5" Ref="U3"  Part="1"
-AR Path="/5D5752FE/5D5C12B5" Ref="U?"  Part="1"
-F 0 "U3" H 4725 3635 50  0000 C CNN
-F 1 "V2164" H 4725 3726 50  0000 C CNN
-F 2 "Package_SO:SOIC-16_3.9x9.9mm_P1.27mm" H 4700 3950 50  0001 C CNN
-F 3 "" H 4700 3950 50  0001 C CNN
-	1    4700 3950
-	1    0    0    1
-$EndComp
 $Comp
 L Device:R R15
@@
 Connection ~ 4300 3950
 Wire Wire Line
-	4300 3950 4400 3950
+	4300 3950 4500 3950
 $Comp
 L Device:R R12
@@
 	5100 3300 5100 2950
 Wire Wire Line
-	5050 3950 5100 3950
-Wire Wire Line
 	5100 3950 5100 3300
 Connection ~ 5100 3300
@@
 $EndComp
 Wire Wire Line
-	4600 4200 6000 4200
-Wire Wire Line
-	6000 4200 6000 3400
+	6000 4250 6000 3400
 Connection ~ 6000 3400
 Wire Wire Line
@@
 	1700 6750 1650 6750
 Connection ~ 1700 6950
+$Comp
+L Schraeg:V2164 U3
+U 1 1 6177084C
+P 4800 3950
+F 0 "U3" H 4800 4318 50  0000 C CNN
+F 1 "V2164" H 4800 4227 50  0000 C CNN
+F 2 "Package_SO:SOIC-16_3.9x9.9mm_P1.27mm" H 4700 4050 50  0001 C CNN
+F 3 "" H 4700 4050 50  0001 C CNN
+	1    4800 3950
+	1    0    0    -1
+$EndComp
+Wire Wire Line
+	4700 4250 6000 4250
 $EndSCHEMATC
