File: Schraeg/power_supply.sch (KiCad schematic (older format))
At the start: 30 parts, among them U1 TL074, U2 TL074, U3 V2164, U4 TL074, U5 TL074

Commit message: Corrected alignment between panel and pcb, changed to slide switches, trimpot for resonance (leaves more space for cutoff) and new panel design.
Parts:
- PWR_IN1: symbol eurocad:EURO_PWR_2x5 -> Schraeg-rescue:EURO_PWR_2x5-eurocad
- U3: symbol v2164:V2164 -> Schraeg-rescue:V2164-v2164
Changed lines of the file:
@@
 EESchema Schematic File Version 4
-LIBS:Schraeg-cache
-EELAYER 26 0
+EELAYER 30 0
 EELAYER END
 $Descr A4 11693 8268
@@
 	2150 3100 2350 3100
 $Comp
-L eurocad:EURO_PWR_2x5 PWR_IN?
+L Schraeg-rescue:EURO_PWR_2x5-eurocad PWR_IN?
 U 1 1 5DA7E2A3
 P 1650 1500
@@
 $EndComp
 $Comp
-L v2164:V2164 U3
+L Schraeg-rescue:V2164-v2164 U3
 U 5 1 5D4D2924
 P 4150 1550
+AR Path="/5D4D2924" Ref="U3"  Part="5"
+AR Path="/5DA7C710/5D4D2924" Ref="U3"  Part="5"
 F 0 "U3" H 4256 1925 50  0000 C CNN
 F 1 "V2164" H 4256 1834 50  0000 C CNN

Commit message: Changed power symbol to generic connector
Parts:
- removed PWR_IN1: EURO_PWR_2x5, Connector_PinHeader_2.54mm:PinHeader_2x05_P2.54mm_Vertical, symbol Schraeg-rescue:EURO_PWR_2x5-eurocad
- added J8: POWER, Connector_PinHeader_2.54mm:PinHeader_2x05_P2.54mm_Vertical, symbol Connector_Generic:Conn_02x05_Odd_Even
- U3: symbol Schraeg-rescue:V2164-v2164 -> Schraeg-rescue:V2164-v2164-Schraeg-rescue
Other:
- moved on the sheet: F1, F2
Changed lines of the file:
@@
 Wire Wire Line
 	2150 3100 2350 3100
-$Comp
-L Schraeg-rescue:EURO_PWR_2x5-eurocad PWR_IN?
-U 1 1 5DA7E2A3
-P 1650 1500
-AR Path="/5DA7E2A3" Ref="PWR_IN?"  Part="1"
-AR Path="/5DA7C710/5DA7E2A3" Ref="PWR_IN1"  Part="1"
-F 0 "PWR_IN1" H 1650 1947 60  0000 C CNN
-F 1 "EURO_PWR_2x5" H 1650 1841 60  0000 C CNN
-F 2 "Connector_PinHeader_2.54mm:PinHeader_2x05_P2.54mm_Vertical" H 1650 1500 60  0001 C CNN
-F 3 "" H 1650 1500 60  0000 C CNN
-	1    1650 1500
-	1    0    0    -1
-$EndComp
-Wire Wire Line
-	1200 1300 1100 1300
-Wire Wire Line
-	1100 1300 1100 1000
-Wire Wire Line
-	1100 1000 1650 1000
+Wire Wire Line
+	1600 1300 1500 1300
+Wire Wire Line
+	1500 1300 1500 1000
+Wire Wire Line
+	1500 1000 1850 1000
 Wire Wire Line
 	2200 1000 2200 1200
@@
 	2200 1300 2100 1300
 Wire Wire Line
-	1200 1700 1100 1700
-Wire Wire Line
-	1100 1700 1100 1900
-Wire Wire Line
-	1100 1900 1650 1900
+	1600 1700 1500 1700
+Wire Wire Line
+	1500 1700 1500 1900
+Wire Wire Line
+	1500 1900 1850 1900
 Wire Wire Line
 	2200 1900 2200 1800
@@
 	2200 1700 2100 1700
 Wire Wire Line
-	1200 1400 1200 1500
-Connection ~ 1200 1500
-Wire Wire Line
-	1200 1500 1200 1600
-Wire Wire Line
-	1200 1500 1000 1500
-Wire Wire Line
-	1000 1500 1000 1600
+	1600 1400 1600 1500
+Connection ~ 1600 1500
+Wire Wire Line
+	1600 1500 1600 1600
+Wire Wire Line
+	1600 1500 1400 1500
+Wire Wire Line
+	1400 1500 1400 1600
 Wire Wire Line
 	2100 1400 2100 1500
@@
 L power:GND #PWR?
 U 1 1 5DA7E2BE
-P 1000 1600
+P 1400 1600
 AR Path="/5DA7E2BE" Ref="#PWR?"  Part="1"
 AR Path="/5DA7C710/5DA7E2BE" Ref="#PWR030"  Part="1"
-F 0 "#PWR030" H 1000 1350 50  0001 C CNN
-F 1 "GND" H 1005 1427 50  0000 C CNN
-F 2 "" H 1000 1600 50  0001 C CNN
-F 3 "" H 1000 1600 50  0001 C CNN
-	1    1000 1600
+F 0 "#PWR030" H 1400 1350 50  0001 C CNN
+F 1 "GND" H 1405 1427 50  0000 C CNN
+F 2 "" H 1400 1600 50  0001 C CNN
+F 3 "" H 1400 1600 50  0001 C CNN
+	1    1400 1600
 	1    0    0    -1
 $EndComp
@@
 L Device:Polyfuse F?
 U 1 1 5DA7E2CA
-P 2550 1200
+P 2550 1800
 AR Path="/5DA7E2CA" Ref="F?"  Part="1"
 AR Path="/5DA7C710/5DA7E2CA" Ref="F1"  Part="1"
-F 0 "F1" V 2325 1200 50  0000 C CNN
-F 1 "Polyfuse" V 2416 1200 50  0000 C CNN
-F 2 "Fuse:Fuse_1206_3216Metric_Pad1.42x1.75mm_HandSolder" H 2600 1000 50  0001 L CNN
-F 3 "~" H 2550 1200 50  0001 C CNN
-	1    2550 1200
+F 0 "F1" V 2325 1800 50  0000 C CNN
+F 1 "Polyfuse" V 2416 1800 50  0000 C CNN
+F 2 "Fuse:Fuse_1206_3216Metric_Pad1.42x1.75mm_HandSolder" H 2600 1600 50  0001 L CNN
+F 3 "~" H 2550 1800 50  0001 C CNN
+	1    2550 1800
 	0    1    1    0
 $EndComp
@@
 L Device:Polyfuse F?
 U 1 1 5DA7E2D8
-P 2550 1800
+P 2550 1200
 AR Path="/5DA7E2D8" Ref="F?"  Part="1"
 AR Path="/5DA7C710/5DA7E2D8" Ref="F2"  Part="1"
-F 0 "F2" V 2325 1800 50  0000 C CNN
-F 1 "Polyfuse" V 2416 1800 50  0000 C CNN
-F 2 "Fuse:Fuse_1206_3216Metric_Pad1.42x1.75mm_HandSolder" H 2600 1600 50  0001 L CNN
-F 3 "~" H 2550 1800 50  0001 C CNN
-	1    2550 1800
+F 0 "F2" V 2325 1200 50  0000 C CNN
+F 1 "Polyfuse" V 2416 1200 50  0000 C CNN
+F 2 "Fuse:Fuse_1206_3216Metric_Pad1.42x1.75mm_HandSolder" H 2600 1000 50  0001 L CNN
+F 3 "~" H 2550 1200 50  0001 C CNN
+	1    2550 1200
 	0    1    1    0
 $EndComp
@@
 L power:PWR_FLAG #FLG?
 U 1 1 5DA7E30D
-P 1650 1000
+P 1850 1000
 AR Path="/5DA7E30D" Ref="#FLG?"  Part="1"
 AR Path="/5DA7C710/5DA7E30D" Ref="#FLG01"  Part="1"
-F 0 "#FLG01" H 1650 1075 50  0001 C CNN
-F 1 "PWR_FLAG" H 1650 1174 50  0000 C CNN
-F 2 "" H 1650 1000 50  0001 C CNN
-F 3 "~" H 1650 1000 50  0001 C CNN
-	1    1650 1000
+F 0 "#FLG01" H 1850 1075 50  0001 C CNN
+F 1 "PWR_FLAG" H 1850 1174 50  0000 C CNN
+F 2 "" H 1850 1000 50  0001 C CNN
+F 3 "~" H 1850 1000 50  0001 C CNN
+	1    1850 1000
 	1    0    0    -1
 $EndComp
@@
 L power:PWR_FLAG #FLG?
 U 1 1 5DA7E314
-P 1650 1900
+P 1850 1900
 AR Path="/5DA7E314" Ref="#FLG?"  Part="1"
 AR Path="/5DA7C710/5DA7E314" Ref="#FLG02"  Part="1"
-F 0 "#FLG02" H 1650 1975 50  0001 C CNN
-F 1 "PWR_FLAG" H 1650 2073 50  0000 C CNN
-F 2 "" H 1650 1900 50  0001 C CNN
-F 3 "~" H 1650 1900 50  0001 C CNN
-	1    1650 1900
+F 0 "#FLG02" H 1850 1975 50  0001 C CNN
+F 1 "PWR_FLAG" H 1850 2073 50  0000 C CNN
+F 2 "" H 1850 1900 50  0001 C CNN
+F 3 "~" H 1850 1900 50  0001 C CNN
+	1    1850 1900
 	-1   0    0    1
 $EndComp
@@
 $EndComp
 $Comp
-L Schraeg-rescue:V2164-v2164 U3
+L Schraeg-rescue:V2164-v2164-Schraeg-rescue U3
 U 5 1 5D4D2924
 P 4150 1550
@@
 Text GLabel 2350 3100 2    50   Input ~ 0
 5V_REF
-Connection ~ 1650 1000
-Wire Wire Line
-	1650 1000 2200 1000
-Connection ~ 1650 1900
-Wire Wire Line
-	1650 1900 2200 1900
+Connection ~ 1850 1000
+Wire Wire Line
+	1850 1000 2200 1000
+Connection ~ 1850 1900
+Wire Wire Line
+	1850 1900 2200 1900
 $Comp
 L power:PWR_FLAG #FLG?
@@
 	0    -1   -1   0
 $EndComp
+$Comp
+L Connector_Generic:Conn_02x05_Odd_Even J8
+U 1 1 616E3FAB
+P 1800 1500
+F 0 "J8" H 1850 1075 50  0000 C CNN
+F 1 "POWER" H 1850 1166 50  0000 C CNN
+F 2 "Connector_PinHeader_2.54mm:PinHeader_2x05_P2.54mm_Vertical" H 1800 1500 50  0001 C CNN
+F 3 "~" H 1800 1500 50  0001 C CNN
+	1    1800 1500
+	1    0    0    1
+$EndComp
 $EndSCHEMATC

Commit message: V2164 symbol in a new library to avoid missing dependencies.
Parts:
- removed U3: V2164, Package_SO:SOIC-16_3.9x9.9mm_P1.27mm, symbol Schraeg-rescue:V2164-v2164-Schraeg-rescue
- added U3: V2164, Package_SO:SOIC-16_3.9x9.9mm_P1.27mm, symbol Schraeg:V2164
Changed lines of the file:
@@
-	1    0    0    -1
-$EndComp
-$Comp
-L Schraeg-rescue:V2164-v2164-Schraeg-rescue U3
-U 5 1 5D4D2924
-P 4150 1550
-AR Path="/5D4D2924" Ref="U3"  Part="5"
-AR Path="/5DA7C710/5D4D2924" Ref="U3"  Part="5"
-F 0 "U3" H 4256 1925 50  0000 C CNN
-F 1 "V2164" H 4256 1834 50  0000 C CNN
-F 2 "Package_SO:SOIC-16_3.9x9.9mm_P1.27mm" H 4150 1550 50  0001 C CNN
-F 3 "" H 4150 1550 50  0001 C CNN
-	5    4150 1550
 	1    0    0    -1
 $EndComp
@@
 	1    0    0    1
 $EndComp
+$Comp
+L Schraeg:V2164 U3
+U 5 1 618650C5
+P 4200 1550
+F 0 "U3" H 4200 1300 50  0000 C CNN
+F 1 "V2164" H 4200 1800 50  0000 C CNN
+F 2 "Package_SO:SOIC-16_3.9x9.9mm_P1.27mm" H 4100 1650 50  0001 C CNN
+F 3 "" H 4100 1650 50  0001 C CNN
+	5    4200 1550
+	-1   0    0    -1
+$EndComp
 $EndSCHEMATC
